File: MutantSMD.kicad_pcb (KiCad board)
At the start: 2 copper layers, 65.3 x 100 mm, 47 parts, among them J1 EURORACK, J2 DC 9V, J3 MATRIX IN, J4 MATRIX OUT, J5 OUT, J6 SYNC IN, J7 SYNC OUT, SW1 FUNC, SW2 TONIC, SW3 SCALE, SW4 START, SW5 REC, SW6 RETRIG, U1 L78M05, U2 MCP6002

Commit message: Mutant SMD v1.0: board text (name, Super-Freq.com, Meebleeps credit), your Dwgs circle; ready for fab
Co-Authored-By: Claude Opus 5.5 <noreply@anthropic.com>
Other:
- board text added: "Mutant SMD v1.0"
- board text added: "Super-Freq.com / Meebleeps"
Changed lines of the file:
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@@
 		)
+	)
+	(gr_circle
+		(center 107.75 124.5)
+		(end 112.75 124.5)
+		(stroke
+			(width 0.1)
+			(type default)
+		)
+		(fill no)
+		(layer "Dwgs.User")
 	)
 	(gr_line
@@
 		(layer "Edge.Cuts")
 	)
+	(gr_text "Super-Freq.com / Meebleeps"
+		(at 113.765999 116 0)
+		(layer "F.SilkS")
+		(effects
+			(font
+				(size 0.9 0.9)
+				(thickness 0.16)
+			)
+		)
+	)
+	(gr_text "Mutant SMD v1.0"
+		(at 113.765999 114.3 0)
+		(layer "F.SilkS")
+		(effects
+			(font
+				(size 1.1 1.1)
+				(thickness 0.16)
+			)
+		)
+	)
 	(segment

Commit message: Matrix supply filter: R8 2R2 + C16 100u tantalum feed the MAX7219 module on its own V5M rail; re-routed; docs, renders
The module's multiplex current pulses no longer modulate the Nano's 5 V (= the D9 audio PWM high level).
Schematic rev 1.0 to match the silkscreen. Adds scripts/pcb_fields.py (LCSC/description fields from the netlist).

Co-Authored-By: Claude Opus 5.5 <noreply@anthropic.com>
Parts:
- added C16: 100u, Capacitor_Tantalum_SMD:CP_EIA-3528-21_Kemet-B, F.Cu at (152.0, 87.6)
- added R8: 2R2, Resistor_SMD:R_1206_3216Metric, F.Cu at (151.6, 107.4)
Connections:
- C10 pad 1: +5V -> /V5M
- C11 pad 1: +5V -> /V5M
- J3 pad 1: +5V -> /V5M
Routing:
- net GND: track 453.2 -> 480.7 mm, vias 0 -> 1
- net /V5M: track 0.00 -> 25.0 mm
- net +5V: track 180.0 -> 191.5 mm, vias 3 -> 4
- net /P2: track 31.1 -> 42.3 mm
- net /P5: track 58.8 -> 49.7 mm
- net /SYNC_IN_D: track 55.8 -> 51.4 mm, vias 0 -> 1
- net Net-(U2A-+): track 16.0 -> 11.9 mm
- net /P4: track 62.8 -> 60.8 mm
- net /SCK: track 39.2 -> 40.5 mm, vias 0 -> 1
- net /V12: track 25.2 -> 26.4 mm
- net /P1: track 26.4 -> 26.3 mm, vias 0 -> 1
