File: MutantSMD.kicad_sch (KiCad schematic)
At the start: 47 parts, among them J1 EURORACK, J2 DC 9V, J3 MATRIX IN, J4 MATRIX OUT, J5 OUT, J6 SYNC IN, J7 SYNC OUT, SW1 FUNC, SW2 TONIC, SW3 SCALE, SW4 START, SW5 REC, SW6 RETRIG, U1 L78M05, U2 MCP6002

Commit message: Add LCSC numbers to all SMD parts; 10u caps to 50 V (C13585), U1 L78M05ABDT-TR (C58069)
Re-linked board footprints to the regenerated schematic; routing unchanged, ERC/DRC/parity clean.

Co-Authored-By: Claude Opus 5.5 <noreply@anthropic.com>
Parts:
- C1, C10, C14, C2: LCSC (none) -> C13585
- C11, C15, C3, C4, C5, C6, C7, C8, C9: LCSC (none) -> C49678
- C12: LCSC (none) -> C1710
- C13: LCSC (none) -> C46653
- R1, R7: LCSC (none) -> C17513
- R2: LCSC (none) -> C17414
- R3, R6: LCSC (none) -> C149504
- R4: LCSC (none) -> C17710
- R5: LCSC (none) -> C17560
- U1: LCSC (none) -> C58069

Commit message: Matrix supply filter: R8 2R2 + C16 100u tantalum feed the MAX7219 module on its own V5M rail; re-routed; docs, renders
The module's multiplex current pulses no longer modulate the Nano's 5 V (= the D9 audio PWM high level).
Schematic rev 1.0 to match the silkscreen. Adds scripts/pcb_fields.py (LCSC/description fields from the netlist).

Co-Authored-By: Claude Opus 5.5 <noreply@anthropic.com>
Parts:
- added C16: 100u, Capacitor_Tantalum_SMD:CP_EIA-3528-21_Kemet-B, symbol Device:C_Polarized
- added R8: 2R2, Resistor_SMD:R_1206_3216Metric, symbol Device:R
Connections:
- net +5V: now also R8.1; no longer C10.1, C11.1, J3.1 (Pin_1)
- net GND: now also C16.2
- new net V5M: C10.1, C11.1, C16.1, J3.1 (Pin_1), R8.2

Commit message: JLC rotation offsets: U2 MCP6002 270, D3 BAT54S 180 (positions regenerated)
Co-Authored-By: Claude Opus 5.5 <noreply@anthropic.com>
Parts:
- D3: FT Rotation Offset (none) -> 180
- U2: FT Rotation Offset (none) -> 270
Changed lines of the file:
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@@
+			)
+		)
+		(property "FT Rotation Offset" "270"
+			(at 365.76 144.78 0)
+			(hide yes)
+			(effects
+				(font
+					(size 1.27 1.27)
+				)
 			)
 		)
@@
 			)
 		)
+		(property "FT Rotation Offset" "270"
+			(at 340.36 177.8 0)
+			(hide yes)
+			(effects
+				(font
+					(size 1.27 1.27)
+				)
+			)
+		)
 		(pin "5"
 		)
@@
 			)
 		)
+		(property "FT Rotation Offset" "270"
+			(at 401.32 177.8 0)
+			(hide yes)
+			(effects
+				(font
+					(size 1.27 1.27)
+				)
+			)
+		)
 		(pin "4"
 		)
@@
 			(at 78.74 233.68 90)
 			(hide yes)
+			(effects
+				(font
+					(size 1.27 1.27)
+				)
+			)
+		)
+		(property "FT Rotation Offset" "180"
+			(at 78.74 233.68 90)
+			(hide yes)
